File: board/PiZeroRobotHat.sch (EAGLE design)
At the start: 31 parts, among them IC1 TPS63061, IC2 MEGA8-AI, J1 AVRISP6_TP, Q1 CSTCR6M00G53Z, U1 DRV8835, U2 PCA9306, X1 1751248, X2 1751248, X3 1751248

Commit message: board improvements
Parts:
- removed C11: 100uF, eagle-ltspice:CC1206
- removed C5: 10uF, rcl:C-EUC0805K
- removed R2: 200K, resistor:R-US_R0603
- removed S1: MOMENTARY-SWITCH-SPST-SMD-RIGHT-ANGLE, SparkFun-Switches:MOMENTARY-SWITCH-SPST-SMD-RIGHT-ANGLE
- removed U2: PCA9306, SparkFun-IC-Comms:PCA9306PCA9306DC-1:1
- added C10, C12, C13: 0.1uF, rcl:C-EUC0603K
- added LD1: PL006-WCR12, led:PL006-WCR12
- added R5: 470k, rcl:R-US_R0603
- added R6: 330k, rcl:R-US_R0603
- added S2: MOMENTARY-SWITCH-SPST-SMD-5.2-REDUNDANT, SparkFun-Switches:MOMENTARY-SWITCH-SPST-SMD-5.2-REDUNDANT
- D1: value 5.6V -> BAT54C; device SparkFun-DiscreteSemi:DIODE-ZENER-MMSZ5232BS -> diode:BAT54C
- JP1: device pinhead:PINHD-1X2/90 -> pinhead:PINHD-1X2
- JP2, JP3: device pinhead:PINHD-1X6/90 -> pinhead:PINHD-1X6
- R3: value 1M -> 10K
- R4: value 10M -> 1M
Connections:
- net N$10 renamed M1A
- net N$6 renamed M0A
- net N$8 renamed M1B
- net N$9 renamed M0B
- removed net 3.3V: U$1.17, U2.VREF1
- removed net N$2: R2.1, U2.EN, U2.VREF2
- removed net SCL1: U$1.5, U2.SCL1
- removed net SCL2: IC2.PC5(ADC5/SCL), U2.SCL2
- removed net SDA1: U$1.3, U2.SDA1
- removed net SDA2: IC2.PC4(ADC4/SDA), U2.SDA2
- new net BUTTON: D1.A1, IC2.PC1(ADC1), LD1.C, R3.1, R4.2
- new net PS_ON: D1.A2, IC2.PC0(ADC0)
- new net SCL: IC2.PC5(ADC5/SCL), U$1.5
- new net SDA: IC2.PC4(ADC4/SDA), U$1.3
- net 5V: now also C10.2, C12.1, C13.1, LED1.A; no longer LED1.C, R2.2
- net ENABLE: now also D1.CC; no longer D1.C, IC2.PC0(ADC0), R4.2, S1.2
- net GND: now also C10.1, C12.2, C13.2, LD1.A, R6.2; no longer C11.2, C5.1, D1.A, U2.GND
- net N$1: now also R3.2, S2.2; no longer R3.1, S1.1
- net N$7: now also LED1.C; no longer LED1.A
- net POWER_GOOD: now also IC2.PC2(ADC2); no longer IC2.PC1(ADC1)
- net VBAT: now also R5.2, R6.1
- net VIN: now also R5.1, S2.1; no longer C11.1, C5.2, R3.2
Other:
- moved on the sheet: J1, JP1, LED1, R3, X1-1, X1-2

Commit message: board improvements
Parts:
- removed U1: DRV8835, bt_motordriver:DRV8835
- removed X2, X3: 1751248, con-phoenix-350:1751248
- added C11, C5: 10uF, rcl:C-EUC0805K
- added C14: 0.1uF, rcl:C-EUC0603K
- added JP4: (no value), pinhead:PINHD-1X3
- added R2: 10K, resistor:R-US_R0603
- added R7: 1M, resistor:R-US_R0603
- added TP1, TP2, TP3: TEST-POINT3X5, SparkFun-Connectors:TEST-POINT3X5
- added U2: DRV8835DSSR, drv8835:DRV8835DSSR
- added X4: 1751264, con-phoenix-350:1751264
Connections:
- new net 0: IC2.PD0(RXD), TP1.1
- new net 1: IC2.PD1(TXD), TP2.1
- new net N$8: IC2.ADC6, TP3.1
- new net SERVO: IC2.PC3(ADC3), JP4.1
- net 5V: now also C5.2, JP4.2, R2.1, U2.VCC; no longer U1.VCC
- net ENABLE: now also C14.2, R7.2
- net EN_A: now also U2.AIN2/AENBL; no longer U1.AIN2/AENBL
- net EN_B: now also U2.BIN2/BENBL; no longer U1.BIN2/BENBL
- net GND: now also C11.1, C14.1, C5.1, JP4.3, R7.1, U2.EPAD, U2.GND; no longer U1.GND1, U1.GND2, U1.PAD1, U1.PAD2, U1.PAD3, U1.PAD4
- net M0A: now also U2.AOUT2, X4-2.K; no longer U1.AOUT2, X2-2.K
- net M0B: now also U2.AOUT1, X4-1.K; no longer U1.AOUT1, X2-1.K
- net M1A: now also U2.BOUT1, X4-3.K; no longer U1.BOUT1, X3-1.K
- net M1B: now also U2.BOUT2, X4-4.K; no longer U1.BOUT2, X3-2.K
- net MODE: now also U2.MODE; no longer U1.MODE
- net PH_A: now also U2.AIN1/APHASE; no longer U1.AIN1/APHASE
- net PH_B: now also U2.BIN1/BPHASE; no longer U1.BIN1/BPHASE
- net RST: now also R2.2
- net VIN: now also C11.2, U2.VM; no longer U1.VM
Other:
- moved on the sheet: C10

Commit message: board improvements
Parts:
- added Q2: (no value), adafruit:MOSFET-NREFLOW
- R3: value 10K -> 1K
- R4, R7: value 1M -> 100K
- S2: value MOMENTARY-SWITCH-SPST-SMD-5.2-REDUNDANT -> MOMENTARY-SWITCH-SPST; device SparkFun-Switches:MOMENTARY-SWITCH-SPST-SMD-5.2-REDUNDANT -> SparkFun-Switches:MOMENTARY-SWITCH-SPST
Connections:
- removed net N$7: LED1.C, R1.1
- new net BT: D1.A1, LD1.C, Q2.G, R3.1, R4.2
- new net N$2: LED1.A, R1.2
- net 5V: now also R1.1; no longer LED1.A
- net BUTTON: now also Q2.D; no longer D1.A1, LD1.C, R3.1, R4.2
- net GND: now also LED1.C, Q2.S; no longer R1.2
Other:
- note added: "Battery voltage divider"
- note added: "Microcontroller"
- note added: "Motor driver"
- note added: "Power input"
- note added: "Power on button"
- note added: "Power supply"
- note added: "Programming header"
- note added: "Raspberry Pi header"
- note added: "Servo connector"
- note added: "Zener 5.1V"
- note removed: "Power supply section"
- moved on the sheet: LED1, R1
